Commit message: Add Foxglove visualization for Lab 3 (Unity/TESSE-style).
Add third-person camera, scene markers, trails via lab3_viz_publisher, foxglove
layout config, and remove RViz. Bridge publishes TF for 3D panel.

File: lab3/gazebo_quadrotor_pkg/urdf/quadrotor.urdf (robot description, URDF)
Before this commit: robot quadrotor, 1 links, 0 joints
Links:
- added link third_person
Joints:
- added joint third_person_joint: type fixed, parent base_link, child third_person, origin xyz=-4.0 0.0 2.5 rpy=0 0.35 0
